File: PCB/Rev2/PH60-SC_Rev2.kicad_pcb (KiCad board)
At the start: 2 copper layers, 285 x 94.6 mm, 219 parts, among them J1 Conn_01x02_Pin, J3 USB_C_Receptacle_USB2.0_14P, J4 Conn_01x02_Pin, U1 nRF52840, X2 32.768kHz, X3 Crystal_Generic

Commit message: Modification of RGB matrix schematic, modification of button matrix schematic, and confirmation of approximate wiring.
Parts:
- added D65: PRTR5V0U2X, Package_TO_SOT_SMD:SOT-143, F.Cu at (47.1, 7.01)
- moved C7 3.17 mm to (184.6, 105.8), turned to 90 degrees
- moved C19 2.28 mm to (169.9, 116.2), turned to 90 degrees
- moved C20 2.11 mm to (169.9, 114.0), turned to 90 degrees
- moved D60 1.70 mm to (271.0, 109.9)
- moved C2 1.63 mm to (179.6, 117.4)
- moved C16 1.34 mm to (175.6, 109.5)
- moved C14 1.29 mm to (188.1, 109.6)
- moved D57 1.22 mm to (152.0, 109.4)
- moved L2 1.15 mm to (178.2, 117.9)
- moved D61 1.01 mm to (295.2, 109.3)
- moved J4 0.89 mm to (188.9, 105.2)
- moved C1 0.89 mm to (173.5, 110.2)
- moved C3 0.86 mm to (175.8, 116.1), turned to -90 degrees
- moved C11 0.80 mm to (187.6, 112.0)
- moved C8 0.80 mm to (189.1, 112.5)
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Connections:
- RGB1 pad 1: VBUS -> rgb_vdd
- RGB1 pad 2: Net-(RGB1-DOUT) -> unconnected-(RGB1-DOUT-Pad2)
- RGB1 pad 4: RGB_IN -> Net-(RGB1-DIN)
- RGB10 pad 1: VBUS -> rgb_vdd
- RGB11 pad 1: VBUS -> rgb_vdd
- RGB11 pad 2: Net-(RGB11-DOUT) -> Net-(RGB10-DIN)
- RGB11 pad 4: Net-(RGB10-DOUT) -> Net-(RGB11-DIN)
- RGB12 pad 1: VBUS -> rgb_vdd
- RGB12 pad 2: Net-(RGB12-DOUT) -> Net-(RGB11-DIN)
- RGB12 pad 4: Net-(RGB11-DOUT) -> Net-(RGB12-DIN)
- RGB13 pad 1: VBUS -> rgb_vdd
- RGB13 pad 2: Net-(RGB13-DOUT) -> Net-(RGB12-DIN)
- RGB13 pad 4: Net-(RGB12-DOUT) -> Net-(RGB13-DIN)
- RGB14 pad 1: VBUS -> rgb_vdd
- RGB14 pad 2: Net-(RGB14-DOUT) -> Net-(RGB13-DIN)
- RGB14 pad 4: Net-(RGB13-DOUT) -> Net-(RGB14-DIN)
- RGB15 pad 1: VBUS -> GND
- RGB15 pad 3: GND -> rgb_vdd
- RGB15 pad 4: Net-(RGB14-DOUT) -> Net-(RGB15-DIN)
- RGB16 pad 1: VBUS -> GND
- RGB16 pad 3: GND -> rgb_vdd
- RGB17 pad 1: VBUS -> GND
- RGB17 pad 3: GND -> rgb_vdd
- RGB18 pad 1: VBUS -> GND
- RGB18 pad 3: GND -> rgb_vdd
- RGB19 pad 1: VBUS -> GND
- RGB19 pad 3: GND -> rgb_vdd
- RGB2 pad 1: VBUS -> rgb_vdd
- RGB2 pad 2: Net-(RGB2-DOUT) -> Net-(RGB1-DIN)
- RGB2 pad 4: Net-(RGB1-DOUT) -> Net-(RGB2-DIN)
- RGB20 pad 1: VBUS -> GND
- RGB20 pad 3: GND -> rgb_vdd
- RGB21 pad 1: VBUS -> GND
- RGB21 pad 3: GND -> rgb_vdd
- RGB22 pad 1: VBUS -> GND
- RGB22 pad 3: GND -> rgb_vdd
- RGB23 pad 1: VBUS -> GND
- RGB23 pad 3: GND -> rgb_vdd
- RGB24 pad 1: VBUS -> GND
- RGB24 pad 3: GND -> rgb_vdd
- RGB25 pad 1: VBUS -> GND
- RGB25 pad 3: GND -> rgb_vdd
- RGB26 pad 1: VBUS -> GND
- RGB26 pad 3: GND -> rgb_vdd
- RGB27 pad 1: VBUS -> GND
- RGB27 pad 3: GND -> rgb_vdd
- RGB28 pad 1: VBUS -> GND
- RGB28 pad 2: Net-(RGB28-DOUT) -> Net-(RGB14-DIN)
- RGB28 pad 3: GND -> rgb_vdd
- RGB29 pad 1: VBUS -> rgb_vdd
- RGB29 pad 2: Net-(RGB29-DOUT) -> Net-(RGB15-DIN)
- RGB29 pad 4: Net-(RGB28-DOUT) -> Net-(RGB29-DIN)
- RGB3 pad 1: VBUS -> rgb_vdd
- RGB3 pad 2: Net-(RGB3-DOUT) -> Net-(RGB2-DIN)
- RGB3 pad 4: Net-(RGB2-DOUT) -> Net-(RGB3-DIN)
- RGB30 pad 1: VBUS -> rgb_vdd
- RGB30 pad 2: Net-(RGB30-DOUT) -> Net-(RGB29-DIN)
- RGB30 pad 4: Net-(RGB29-DOUT) -> Net-(RGB30-DIN)
- RGB31 pad 1: VBUS -> rgb_vdd
- RGB31 pad 2: Net-(RGB31-DOUT) -> Net-(RGB30-DIN)
- RGB31 pad 4: Net-(RGB30-DOUT) -> Net-(RGB31-DIN)
- RGB32 pad 1: VBUS -> rgb_vdd
- RGB32 pad 2: Net-(RGB32-DOUT) -> Net-(RGB31-DIN)
- RGB32 pad 4: Net-(RGB31-DOUT) -> Net-(RGB32-DIN)
- RGB33 pad 1: VBUS -> rgb_vdd
- RGB33 pad 2: Net-(RGB33-DOUT) -> Net-(RGB32-DIN)
- RGB33 pad 4: Net-(RGB32-DOUT) -> Net-(RGB33-DIN)
- RGB34 pad 1: VBUS -> rgb_vdd
- RGB34 pad 2: Net-(RGB34-DOUT) -> Net-(RGB33-DIN)
- RGB34 pad 4: Net-(RGB33-DOUT) -> Net-(RGB34-DIN)
- RGB35 pad 1: VBUS -> rgb_vdd
- RGB35 pad 2: Net-(RGB35-DOUT) -> Net-(RGB34-DIN)
- RGB35 pad 4: Net-(RGB34-DOUT) -> Net-(RGB35-DIN)
- RGB36 pad 1: VBUS -> rgb_vdd
- RGB36 pad 2: Net-(RGB36-DOUT) -> Net-(RGB35-DIN)
- RGB36 pad 4: Net-(RGB35-DOUT) -> Net-(RGB36-DIN)
- RGB37 pad 1: VBUS -> rgb_vdd
- RGB37 pad 2: Net-(RGB37-DOUT) -> Net-(RGB36-DIN)
- RGB37 pad 4: Net-(RGB36-DOUT) -> Net-(RGB37-DIN)
- RGB38 pad 1: VBUS -> rgb_vdd
- RGB38 pad 2: Net-(RGB38-DOUT) -> Net-(RGB37-DIN)
- RGB38 pad 4: Net-(RGB37-DOUT) -> Net-(RGB38-DIN)
- RGB39 pad 1: VBUS -> rgb_vdd
- RGB39 pad 2: Net-(RGB39-DOUT) -> Net-(RGB38-DIN)
- RGB39 pad 4: Net-(RGB38-DOUT) -> Net-(RGB39-DIN)
- RGB4 pad 1: VBUS -> rgb_vdd
- RGB4 pad 2: Net-(RGB4-DOUT) -> Net-(RGB3-DIN)
- RGB4 pad 4: Net-(RGB3-DOUT) -> Net-(RGB4-DIN)
- RGB40 pad 1: VBUS -> rgb_vdd
- RGB40 pad 2: Net-(RGB40-DOUT) -> Net-(RGB39-DIN)
- RGB40 pad 4: Net-(RGB39-DOUT) -> Net-(RGB40-DIN)
- RGB41 pad 1: VBUS -> rgb_vdd
- RGB41 pad 2: Net-(RGB41-DOUT) -> Net-(RGB40-DIN)
- RGB41 pad 4: Net-(RGB40-DOUT) -> Net-(RGB41-DIN)
- RGB42 pad 1: VBUS -> rgb_vdd
- RGB42 pad 4: Net-(RGB41-DOUT) -> Net-(RGB42-DIN)
- RGB43 pad 1: VBUS -> rgb_vdd
- RGB44 pad 1: VBUS -> rgb_vdd
- RGB45 pad 1: VBUS -> rgb_vdd
- RGB46 pad 1: VBUS -> rgb_vdd
- RGB47 pad 1: VBUS -> rgb_vdd
- RGB48 pad 1: VBUS -> rgb_vdd
- RGB49 pad 1: VBUS -> rgb_vdd
- RGB5 pad 1: VBUS -> rgb_vdd
- RGB5 pad 2: Net-(RGB5-DOUT) -> Net-(RGB4-DIN)
- RGB5 pad 4: Net-(RGB4-DOUT) -> Net-(RGB5-DIN)
- RGB50 pad 1: VBUS -> rgb_vdd
- RGB51 pad 1: VBUS -> rgb_vdd
- RGB52 pad 1: VBUS -> rgb_vdd
- RGB53 pad 1: VBUS -> rgb_vdd
- RGB53 pad 2: Net-(RGB53-DOUT) -> Net-(RGB41-DIN)
- RGB54 pad 1: VBUS -> rgb_vdd
- RGB54 pad 2: Net-(RGB54-DOUT) -> Net-(RGB42-DIN)
- RGB54 pad 4: Net-(RGB53-DOUT) -> Net-(RGB54-DIN)
- RGB55 pad 1: VBUS -> rgb_vdd
- RGB55 pad 2: Net-(RGB55-DOUT) -> Net-(RGB54-DIN)
- RGB55 pad 4: Net-(RGB54-DOUT) -> Net-(RGB55-DIN)
- RGB56 pad 1: VBUS -> rgb_vdd
- RGB56 pad 2: Net-(RGB56-DOUT) -> Net-(RGB55-DIN)
- RGB56 pad 4: Net-(RGB55-DOUT) -> Net-(RGB56-DIN)
- RGB57 pad 1: VBUS -> rgb_vdd
- RGB57 pad 2: Net-(RGB57-DOUT) -> Net-(RGB56-DIN)
- RGB57 pad 4: Net-(RGB56-DOUT) -> Net-(RGB57-DIN)
- RGB58 pad 1: VBUS -> rgb_vdd
- RGB58 pad 2: Net-(RGB58-DOUT) -> Net-(RGB57-DIN)
- RGB58 pad 4: Net-(RGB57-DOUT) -> Net-(RGB58-DIN)
- RGB59 pad 1: VBUS -> rgb_vdd
- RGB59 pad 2: Net-(RGB59-DOUT) -> Net-(RGB58-DIN)
- RGB59 pad 4: Net-(RGB58-DOUT) -> Net-(RGB59-DIN)
- RGB6 pad 1: VBUS -> rgb_vdd
- RGB6 pad 2: Net-(RGB6-DOUT) -> Net-(RGB5-DIN)
- RGB6 pad 4: Net-(RGB5-DOUT) -> Net-(RGB6-DIN)
- RGB60 pad 1: VBUS -> rgb_vdd
- RGB60 pad 2: Net-(RGB60-DOUT) -> Net-(RGB59-DIN)
- RGB60 pad 4: Net-(RGB59-DOUT) -> Net-(RGB60-DIN)
- RGB61 pad 1: VBUS -> rgb_vdd
- RGB61 pad 2: unconnected-(RGB61-DOUT-Pad2) -> Net-(RGB60-DIN)
- RGB61 pad 4: Net-(RGB60-DOUT) -> RGB_IN
- RGB7 pad 1: VBUS -> rgb_vdd
- RGB7 pad 2: Net-(RGB7-DOUT) -> Net-(RGB6-DIN)
- RGB7 pad 4: Net-(RGB6-DOUT) -> Net-(RGB7-DIN)
- RGB8 pad 1: VBUS -> rgb_vdd
- RGB8 pad 2: Net-(RGB8-DOUT) -> Net-(RGB7-DIN)
- RGB8 pad 4: Net-(RGB7-DOUT) -> Net-(RGB8-DIN)
- RGB9 pad 1: VBUS -> rgb_vdd
- RGB9 pad 2: Net-(RGB10-DIN) -> Net-(RGB8-DIN)
- RGB9 pad 4: Net-(RGB8-DOUT) -> Net-(RGB10-DOUT)
- U1 pad A10: col_1 -> unconnected-(U1-AIN5/P0.29-PadA10)
- U1 pad A12: row_4 -> unconnected-(U1-AIN0/P0.02-PadA12)
- U1 pad A8: col_2 -> unconnected-(U1-AIN7/P0.31-PadA8)
- U1 pad AC15: col_6 -> unconnected-(U1-P0.19-PadAC15)
- U1 pad AC17: col_8 -> unconnected-(U1-P0.21-PadAC17)
- U1 pad AC19: col_10 -> unconnected-(U1-P0.23-PadAC19)
- U1 pad AC21: col_12 -> row_4
- U1 pad G1: RGB_IN -> col_1
- U1 pad J1: unconnected-(U1-AIN2/P0.04-PadJ1) -> col_6
- U1 pad L24: unconnected-(U1-NFC1/P0.09-PadL24) -> col_10
- U1 pad R24: unconnected-(U1-P1.06-PadR24) -> col_12
- U1 pad T2: unconnected-(U1-TRACEDATA2/P0.11-PadT2) -> col_2
- U1 pad U24: unconnected-(U1-P1.04-PadU24) -> col_8
- U1 pad W24: unconnected-(U1-P1.02-PadW24) -> RGB_IN
Routing:
- net row_3: track 31.0 -> 273.9 mm, vias 0 -> 2
- net col_1: track 0.00 -> 202.9 mm, vias 0 -> 3
- net col_13: track 0.00 -> 198.9 mm, vias 0 -> 1
- net col_0: track 65.7 -> 229.2 mm, vias 0 -> 3
- net col_12: track 65.7 -> 203.4 mm, vias 0 -> 3
- net row_1: track 200.0 -> 333.1 mm, vias 0 -> 2
- net row_4: track 142.9 -> 272.3 mm, vias 0 -> 3
- net RGB_IN: track 0.00 -> 124.4 mm
- net col_2: track 65.7 -> 186.1 mm, vias 0 -> 3
- net row_0: track 257.2 -> 355.3 mm, vias 0 -> 2
- net col_11: track 65.7 -> 161.7 mm
- net col_3: track 65.7 -> 149.2 mm
- net col_10: track 65.7 -> 138.7 mm, vias 0 -> 1
- net col_4: track 65.7 -> 130.7 mm
- net row_2: track 247.7 -> 303.1 mm, vias 0 -> 2
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- added copper zone on B.Cu, net RGB_IN
- removed copper zone on B.Cu, net (none)
- removed copper zone on B.Cu, net GND
- removed copper zone on F.Cu, net GND
- removed copper zone on B.Cu, net VBUS
- removed copper zone on F.Cu, net VBUS

Commit message: The basic layout is complete, and a full DRC scan is underway. RGB signal line interference needs to be considered. The battery connector has not yet been selected.
Parts:
- added Q3: 2N7002, PCM_Package_TO_SOT_SMD_AKL:SOT-23, B.Cu at (274.4, 72.7)
- added Q4: BSS84, PCM_Package_TO_SOT_SMD_AKL:SOT-23, B.Cu at (272.1, 77.2)
- added R2: 100K, PCM_Resistor_SMD_AKL:R_0603_1608Metric_Pad1.05x0.95mm, B.Cu at (267.4, 78.8)
- D65: moved to B.Cu
- moved D65 56.7 mm to (53.4, 63.4), turned to -90 degrees
- moved J3 50.0 mm to (31.3, 70.5), turned to 90 degrees
- moved R5 38.2 mm to (36.8, 74.3)
- moved R6 29.7 mm to (36.8, 64.5), turned to 90 degrees
- moved D42 25.1 mm to (68.1, 89.3)
- moved D53 19.6 mm to (261.5, 89.0)
- moved D14 12.8 mm to (275.5, 31.9)
- moved RGB41 7.55 mm to (287.0, 75.6), turned to -90 degrees
- moved RGB53 7.52 mm to (282.5, 94.9), turned to -90 degrees
- moved RGB28 7.52 mm to (294.4, 56.8), turned to -90 degrees
- moved RGB42 7.52 mm to (44.3, 94.9), turned to -90 degrees
- moved RGB14 7.50 mm to (289.9, 38.0), turned to -90 degrees
- moved C18 3.64 mm to (173.6, 106.5), turned to 90 degrees
- moved D41 3.57 mm to (287.9, 67.3), turned to 0 degrees
- moved D28 2.58 mm to (294.6, 49.1), turned to 0 degrees
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Connections:
- U1 pad AC15: unconnected-(U1-P0.19-PadAC15) -> RGB_SW
- U1 pad AC21: row_4 -> col_1
- U1 pad G1: col_1 -> row_4
Routing:
- net rgb_vdd: track 0.00 -> 916.0 mm, vias 0 -> 141
- net /USB_D+: track 0.85 -> 217.7 mm, vias 1 -> 4
- net /USB_D-: track 0.77 -> 214.8 mm, vias 1 -> 4
- net RGB_SW: track 0.00 -> 123.6 mm, vias 0 -> 2
- net Net-(RGB57-DIN): track 0.00 -> 79.1 mm, vias 0 -> 2
- net Net-(RGB56-DIN): track 1.41 -> 73.4 mm
- net row_3: track 273.9 -> 229.3 mm
- net /RESET: track 0.00 -> 39.6 mm, vias 0 -> 3
- net Net-(D53-A): track 8.50 -> 41.9 mm
- net Net-(D14-A): track 8.29 -> 35.6 mm, vias 0 -> 2
- net col_13: track 198.9 -> 219.9 mm, vias 1 -> 0
- net Net-(D42-A): track 8.50 -> 26.9 mm
- net Net-(RGB42-DOUT): track 26.7 -> 41.4 mm
- net GND: track 2.48 -> 16.1 mm, vias 1 -> 369
- net VBUS: track 5.81 -> 18.9 mm, vias 0 -> 30
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- added copper zone on B.Cu, net GND
- added copper zone on F.Cu, net GND
- added copper zone on B.Cu, net Net-(Q3-S)
- added copper zone on B.Cu, net VBUS
- added copper zone on F.Cu, net VBUS
- added copper zone on B.Cu, net rgb_vdd
- added copper zone on F.Cu, net rgb_vdd
- removed copper zone on F.Cu, net (none)
- removed copper zone on B.Cu, net RGB_IN
Other:
- outline, holes or cut-outs redrawn

Commit message: layout
Parts:
- added C21: 12p, Capacitor_SMD:C_0402_1005Metric, B.Cu at (271.9, 80.5)
- added C22: 100p, Capacitor_SMD:C_0402_1005Metric, B.Cu at (37.7, 47.1)
- added C23: 100p, Capacitor_SMD:C_0402_1005Metric, B.Cu at (37.8, 85.6)
Routing:
- net GND: track 16.1 -> 19.0 mm, vias 369 -> 468
- net col_10: track 138.0 -> 139.8 mm
- net rgb_vdd: track 916.0 -> 914.4 mm
- net col_12: track 207.3 -> 206.2 mm
