File: PCB/Rev2/PH60-SC_Rev2.kicad_pcb (KiCad board)
At the start: 2 copper layers, 285 x 94.6 mm, 226 parts, among them J1 Conn_01x02_Pin, J3 USB_C_Receptacle_USB2.0_14P, J4 Conn_01x02_Pin, Q3 2N7002, Q4 BSS84, U1 nRF52840, X2 32.768kHz, X3 Crystal_Generic

Commit message: layout
Parts:
- moved D28 0.50 mm to (294.1, 49.1)
Changed lines of the file:
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@@
 	(footprint "Diode_SMD:D_SOD-123"
 		(layer "B.Cu")
-		(at 294.575 49.075)
+		(at 294.075 49.075)
 		(descr "SOD-123")
 		(tags "SOD-123")
@@
 	)
 	(segment
-		(start 35.862501 49.5)
-		(end 293.037501 49.5)
+		(start 177.848224 110.535)
+		(end 178.025 110.535)
 		(width 0.2)
 		(layer "B.Cu")
@@
 	)
 	(segment
-		(start 177.848224 110.535)
-		(end 178.025 110.535)
+		(start 177.5092 110.575)
+		(end 177.808224 110.575)
 		(width 0.2)
 		(layer "B.Cu")
@@
 	)
 	(segment
-		(start 177.5092 110.575)
-		(end 177.808224 110.575)
+		(start 35.887501 49.475)
+		(end 292.025 49.475)
 		(width 0.2)
 		(layer "B.Cu")
@@
 	)
 	(segment
+		(start 292.025 49.475)
+		(end 292.425 49.075)
+		(width 0.2)
+		(layer "B.Cu")
+		(net 23)
+	)
+	(segment
+		(start 35.862501 49.5)
+		(end 35.887501 49.475)
+		(width 0.2)
+		(layer "B.Cu")
+		(net 23)
+	)
+	(segment
 		(start 170.257 111.487)
 		(end 176.5972 111.487)
@@
 	)
 	(segment
-		(start 296.225 49.075)
-		(end 296.225 49.675)
-		(width 0.2)
-		(layer "B.Cu")
-		(net 36)
-	)
-	(segment
-		(start 303.47 55.923237)
-		(end 303.47 61.7925)
-		(width 0.2)
-		(layer "B.Cu")
-		(net 36)
-	)
-	(segment
-		(start 296.175 49.725)
-		(end 296.175 50.875)
+		(start 299.975 52.975)
+		(end 303.47 56.47)
 		(width 0.2)
 		(layer "B.Cu")
@@
 	)
 	(segment
-		(start 300.521763 52.975)
-		(end 303.47 55.923237)
+		(start 295.725 49.075)
+		(end 295.725 50.025)
 		(width 0.2)
 		(layer "B.Cu")
@@
 	)
 	(segment
-		(start 296.225 49.675)
-		(end 296.175 49.725)
+		(start 295.725 50.025)
+		(end 298.675 52.975)
 		(width 0.2)
 		(layer "B.Cu")
@@
 	)
 	(segment
-		(start 298.275 52.975)
-		(end 300.521763 52.975)
+		(start 303.47 56.47)
+		(end 303.47 61.7925)
 		(width 0.2)
 		(layer "B.Cu")
@@
 	)
 	(segment
-		(start 296.175 50.875)
-		(end 298.275 52.975)
+		(start 298.675 52.975)
+		(end 299.975 52.975)
 		(width 0.2)
 		(layer "B.Cu")

Commit message: layout and drc
Parts:
- moved C20 2.90 mm to (167.0, 114.1)
- moved X2 2.90 mm to (168.8, 115.2)
- moved C19 2.80 mm to (167.1, 116.2)
- moved D14 0.94 mm to (275.8, 31.0), turned to 0 degrees
- moved C16 0.41 mm to (175.2, 109.6)
- moved C22 0.13 mm to (37.6, 47.1)
Connections:
- U1 pad AC21: col_1 -> unconnected-(U1-P0.25-PadAC21)
- U1 pad B11: unconnected-(U1-AIN4/P0.28-PadB11) -> col_1
Routing:
- net row_4: track 278.0 -> 299.7 mm, vias 3 -> 5
- net VDD_Output: track 63.0 -> 55.7 mm
- net col_1: track 207.9 -> 203.2 mm
- net Net-(U1-XL1/P0.00): track 10.2 -> 13.7 mm
- net Net-(U1-XL2/P0.01): track 10.7 -> 13.8 mm
- net rgb_vdd: track 914.4 -> 912.8 mm, vias 141 -> 142
- net Net-(RGB13-DIN): track 22.8 -> 24.3 mm
- net col_0: track 224.9 -> 226.2 mm, vias 4 -> 3
- net col_8: track 83.8 -> 82.5 mm
- net Net-(D29-A): track 8.50 -> 7.30 mm
- net Net-(RGB57-DIN): track 79.1 -> 80.3 mm
- net GND: track 19.0 -> 20.0 mm, vias 468 -> 522
- net VBUS: track 18.9 -> 19.9 mm
- net Net-(RGB52-DOUT): track 40.0 -> 39.1 mm
- net col_13: track 219.9 -> 219.2 mm
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Other:
- outline, holes or cut-outs redrawn
