File: PCB/Rev2.1/matrix.kicad_sch (KiCad schematic)
At the start: 127 parts

Commit message: 布局调整，rgb，轴座调整，注意二极管位置为手动校准
Parts:
- removed ST4: choc_stab, STAB:STAB_CHOC_2U, symbol PCM_marbastlib-choc:choc_stab
- added D43: DIODE, Diode_SMD:D_SOD-123, symbol Device:D
- added S54: Choc_V2, PH60:SW_Hotswap_Kailh_Choc_V2_Plated_Nosilkscreen, symbol Switch:SW_Push
- renumbered D43 to D44, D44 to D45, D45 to D46, D46 to D47, D47 to D48, D48 to D49, D49 to D50, D50 to D51, D51 to D52, D52 to D53, D53 to D54, D54 to D55, D55 to D56, D56 to D57, D57 to D58, D58 to D59, D59 to D60, D60 to D61, D61 to D62, D62 to D63, S54 to S55, S55 to S56, S56 to S57, S57 to S58, S58 to S59, S59 to S60, S60 to S61, S61 to S62, ST5 to ST1, ST1 to ST2, ST2 to ST3, ST3 to ST4
Connections:
- net col_13: now also S54.1
- net row_3: now also D43.1 (K)
- new net: D43.2 (A), S54.2
