File: PCB/Rev2.1/battery.kicad_sch (KiCad schematic)
At the start: 11 parts, among them U2 TP4057, U3 TPS2116DRL, U4 TPS2116DRL

Commit message: Delete resistor and route
Connections:
- net BATT_STAT: no longer names the net of U4.8 (ST)
- no-connect marks 3 -> 4
Changed lines of the file:
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@@
+	)
+	(no_connect
+		(at 181.61 101.6)
 	)
 	(no_connect
@@
 			)
 		)
-	)
-	(global_label "BATT_STAT"
-		(shape input)
-		(at 181.61 101.6 0)
-		(fields_autoplaced yes)
-		(effects
-			(font
-				(size 1.27 1.27)
-			)
-			(justify left)
-		)
-		(property "Intersheetrefs" "${INTERSHEET_REFS}"
-			(at 194.0899 101.6 0)
-			(hide yes)
-			(show_name no)
-			(do_not_autoplace no)
-			(effects
-				(font
-					(size 1.27 1.27)
-				)
-				(justify left)
-			)
-		)
